File: solder.kicad_pcb (KiCad board)
At the start: 2 copper layers, 93.8 x 65 mm, 34 parts, among them Q1 2N3904

Commit message: pcb and gerber in prod
Parts:
- added G***: LOGO, kicadlogos:rtx, B.Cu at (82.5, 93.5)
- added G*** (x2): LOGO, LOGO, F.Cu at (86.0, 93.5)
- added G***: LOGO, kicadlogos:India, F.Cu at (133.0, 70.0)
- BT1, BT2: footprint Battery:BatteryHolder_Keystone_1060_1x2032 -> Battery:BatteryHolder_Keystone_3034_1x20mm
- R3: moved to B.Cu
- moved R3 7.23 mm to (102.5, 91.5), turned to -90 degrees
- moved RV1 1.42 mm to (99.9, 90.4)
Routing:
- net +5V: track 16.1 -> 50.2 mm
- net Net-(Q1-B): track 45.4 -> 79.3 mm
- net GND: track 75.7 -> 74.1 mm
Other:
- board text added: "Souptik Samanta"
