File: solder.kicad_sch (KiCad schematic)
At the start: 18 parts, among them M1 Motor_DC, Q1 2N3904

Commit message: pcb and gerber in prod
Parts:
- BT1, BT2: footprint Battery:BatteryHolder_Keystone_1060_1x2032 -> Battery:BatteryHolder_Keystone_3034_1x20mm
Changed lines of the file:
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@@
 			)
 		)
-		(property "Footprint" "Battery:BatteryHolder_Keystone_1060_1x2032"
+		(property "Footprint" "Battery:BatteryHolder_Keystone_3034_1x20mm"
 			(at 27.94 103.886 90)
 			(effects
@@
 			)
 		)
-		(property "Footprint" "Battery:BatteryHolder_Keystone_1060_1x2032"
+		(property "Footprint" "Battery:BatteryHolder_Keystone_3034_1x20mm"
 			(at 40.64 103.886 90)
 			(effects
